Commit message: new name and correct position markers

File: tactile_glove_display/urdf/puthand-standalone.urdf.xacro (robot description, xacro)
@@ -2,6 +2,6 @@
 <robot name="puthand" xmlns:xacro="http://ros.org/wiki/xacro">
  <!-- common stuff -->
- <xacro:include filename="$(find tactile_glove)/urdf/common.gazebo.xacro" />
- <xacro:include filename="$(find tactile_glove)/urdf/puthand.urdf.xacro" />
+ <xacro:include filename="$(find tactile_glove_display)/urdf/common.gazebo.xacro" />
+ <xacro:include filename="$(find tactile_glove_display)/urdf/puthand.urdf.xacro" />
  <link name="base_link" />
  <xacro:puthand parent="base_link" name="left_hand" prefix="">

File: tactile_glove_display/urdf/puthand.urdf.xacro (robot description, xacro)
@@ -1,6 +1,6 @@
 <?xml version="1.0"?>
 <robot xmlns:xacro="http://ros.org/wiki/xacro">
-  <xacro:include filename="$(find tactile_glove)/urdf/puthand.transmission.xacro" />
-  <xacro:include filename="$(find tactile_glove)/urdf/puthand.gazebo.xacro" />
+  <xacro:include filename="$(find tactile_glove_display)/urdf/puthand.transmission.xacro" />
+  <xacro:include filename="$(find tactile_glove_display)/urdf/puthand.gazebo.xacro" />
   <xacro:property name="cyl_radius" value="0.001" />
   <!-- Inertia parameters -->
@@ -40,5 +40,5 @@
 	<origin xyz="0 0 0.0" rpy="0 0 0" />
 	<geometry>
-          <mesh filename="package://tactile_glove/meshes/metacarpusNew.dae" />
+          <mesh filename="package://tactile_glove_display/meshes/metacarpusNew.dae" />
 	</geometry>
       </visual>
@@ -46,5 +46,5 @@
 	<origin xyz="0 0 0.0" rpy="0 0 0" />
 	<geometry>
-          <mesh filename="package://tactile_glove/meshes/metacarpusNew.dae" />
+          <mesh filename="package://tactile_glove_display/meshes/metacarpusNew.dae" />
 	</geometry>
       </collision>
@@ -58,5 +58,5 @@
 	<origin xyz="0 0 0" rpy="0 0 0" />
 	<geometry>
-          <mesh filename="package://tactile_glove/meshes/metacarpal.dae" />
+          <mesh filename="package://tactile_glove_display/meshes/metacarpal.dae" />
 	</geometry>
       </visual>
@@ -64,5 +64,5 @@
 	<origin xyz="0 0 0" rpy="0 0 0" />
 	<geometry>
-          <mesh filename="package://tactile_glove/meshes/metacarpal.dae" />
+          <mesh filename="package://tactile_glove_display/meshes/metacarpal.dae" />
 	</geometry>
       </collision>
@@ -75,5 +75,5 @@
 	<origin xyz="0 0 0" rpy="0 0 0" />
 	<geometry>
-          <mesh filename="package://tactile_glove/meshes/thumbProximal.dae" />
+          <mesh filename="package://tactile_glove_display/meshes/thumbProximal.dae" />
 	</geometry>
       </visual>
@@ -81,5 +81,5 @@
           <origin xyz="0 0 0" rpy="0 0 0" />
 	<geometry>
-          <mesh filename="package://tactile_glove/meshes/thumbProximal.dae" />
+          <mesh filename="package://tactile_glove_display/meshes/thumbProximal.dae" />
 	</geometry>
       </collision>
@@ -92,5 +92,5 @@
 	<origin xyz="0 0 0" rpy="0 0 -1.5708" />
 	<geometry>
-          <mesh filename="package://tactile_glove/meshes/thumbDistal.dae" />
+          <mesh filename="package://tactile_glove_display/meshes/thumbDistal.dae" />
 	</geometry>
       </visual>
@@ -98,5 +98,5 @@
           <origin xyz="0 0 0" rpy="0 0 -1.5708" />
 	<geometry>
-          <mesh filename="package://tactile_glove/meshes/thumbDistal.dae" />
+          <mesh filename="package://tactile_glove_display/meshes/thumbDistal.dae" />
 	</geometry>
       </collision>
@@ -149,11 +149,11 @@
 	<origin xyz="-0.00 -0.00 0.00" rpy="0 0 0" />
 	<geometry>
-          <mesh filename="package://tactile_glove/meshes/fingerProximal.dae" />
-	</geometry>
-      </visual>
-      <collision>
-	<origin xyz="-0.00 -0.00 0.00" rpy="0 0 0" />
-	<geometry>
-          <mesh filename="package://tactile_glove/meshes/fingerProximal.dae" />
+          <mesh filename="package://tactile_glove_display/meshes/fingerProximal.dae" />
+	</geometry>
+      </visual>
+      <collision>
+	<origin xyz="-0.00 -0.00 0.00" rpy="0 0 0" />
+	<geometry>
+          <mesh filename="package://tactile_glove_display/meshes/fingerProximal.dae" />
 	</geometry>
       </collision>
@@ -166,5 +166,5 @@
 	<origin xyz="-0.00 -0.00 0.00" rpy="0 0 1.5708" />
 	<geometry>
-          <mesh filename="package://tactile_glove/meshes/fingerMiddle.dae" />
+          <mesh filename="package://tactile_glove_display/meshes/fingerMiddle.dae" />
 	</geometry>
       </visual>
@@ -172,5 +172,5 @@
           <origin xyz="-0.00 -0.00 0.00" rpy="0 0 1.5708" />
 	<geometry>
-          <mesh filename="package://tactile_glove/meshes/fingerMiddle.dae" />
+          <mesh filename="package://tactile_glove_display/meshes/fingerMiddle.dae" />
 	</geometry>
       </collision>
@@ -183,5 +183,5 @@
 	<origin xyz="-0.00 -0.00 0.00" rpy="0 0 0" />
 	<geometry>
-          <mesh filename="package://tactile_glove/meshes/fingerDistal.dae" />
+          <mesh filename="package://tactile_glove_display/meshes/fingerDistal.dae" />
 	</geometry>
       </visual>
@@ -189,5 +189,5 @@
           <origin xyz="-0.00 -0.0 0.00" rpy="0 0 0" />
 	<geometry>
-          <mesh filename="package://tactile_glove/meshes/fingerDistal.dae" />
+          <mesh filename="package://tactile_glove_display/meshes/fingerDistal.dae" />
 	</geometry>
       </collision>
@@ -240,11 +240,11 @@
 	<origin xyz="-0.00 -0.00 0.00" rpy="0 0 0" />
 	<geometry>
-          <mesh filename="package://tactile_glove/meshes/fingerProximal.dae" />
-	</geometry>
-      </visual>
-      <collision>
-	<origin xyz="-0.00 -0.00 0.00" rpy="0 0 0" />
-	<geometry>
-          <mesh filename="package://tactile_glove/meshes/fingerProximal.dae" />
+          <mesh filename="package://tactile_glove_display/meshes/fingerProximal.dae" />
+	</geometry>
+      </visual>
+      <collision>
+	<origin xyz="-0.00 -0.00 0.00" rpy="0 0 0" />
+	<geometry>
+          <mesh filename="package://tactile_glove_display/meshes/fingerProximal.dae" />
 	</geometry>
       </collision>
@@ -257,5 +257,5 @@
 	<origin xyz="-0.00 -0.00 0.00" rpy="0 0 1.5708" />
 	<geometry>
-          <mesh filename="package://tactile_glove/meshes/fingerMiddle.dae" />
+          <mesh filename="package://tactile_glove_display/meshes/fingerMiddle.dae" />
 	</geometry>
       </visual>
@@ -263,5 +263,5 @@
           <origin xyz="-0.00 -0.00 0.00" rpy="0 0 1.5708" />
 	<geometry>
-          <mesh filename="package://tactile_glove/meshes/fingerMiddle.dae" />
+          <mesh filename="package://tactile_glove_display/meshes/fingerMiddle.dae" />
 	</geometry>
       </collision>
@@ -274,5 +274,5 @@
 	<origin xyz="-0.00 -0.00 0.00" rpy="0 0 0" />
 	<geometry>
-          <mesh filename="package://tactile_glove/meshes/fingerDistal.dae" />
+          <mesh filename="package://tactile_glove_display/meshes/fingerDistal.dae" />
 	</geometry>
       </visual>
@@ -280,5 +280,5 @@
           <origin xyz="-0.00 -0.00 0.00" rpy="0 0 0" />
 	<geometry>
-          <mesh filename="package://tactile_glove/meshes/fingerDistal.dae" />
+          <mesh filename="package://tactile_glove_display/meshes/fingerDistal.dae" />
 	</geometry>
       </collision>
@@ -328,11 +328,11 @@
 	<origin xyz="-0.00 -0.00 0.00" rpy="0 0 0" />
 	<geometry>
-          <mesh filename="package://tactile_glove/meshes/f4phalanx1.dae" />
-	</geometry>
-      </visual>
-      <collision>
-	<origin xyz="-0.00 -0.00 0.00" rpy="0 0 0" />
-	<geometry>
-          <mesh filename="package://tactile_glove/meshes/f4phalanx1.dae" />
+          <mesh filename="package://tactile_glove_display/meshes/f4phalanx1.dae" />
+	</geometry>
+      </visual>
+      <collision>
+	<origin xyz="-0.00 -0.00 0.00" rpy="0 0 0" />
+	<geometry>
+          <mesh filename="package://tactile_glove_display/meshes/f4phalanx1.dae" />
 	</geometry>
       </collision>
@@ -345,5 +345,5 @@
 	<origin xyz="-0.00 -0.00 0.00" rpy="0 0 0" />
 	<geometry>
-          <mesh filename="package://tactile_glove/meshes/f4phalanx2.dae" />
+          <mesh filename="package://tactile_glove_display/meshes/f4phalanx2.dae" />
 	</geometry>
       </visual>
@@ -351,5 +351,5 @@
           <origin xyz="-0.00 -0.00 0.00" rpy="0 0 0" />
 	<geometry>
-          <mesh filename="package://tactile_glove/meshes/f4phalanx2.dae" />
+          <mesh filename="package://tactile_glove_display/meshes/f4phalanx2.dae" />
 	</geometry>
       </collision>
@@ -362,5 +362,5 @@
 	<origin xyz="-0.00 -0.00 0.00" rpy="0 0 0" />
 	<geometry>
-          <mesh filename="package://tactile_glove/meshes/f45phalanx3.dae" />
+          <mesh filename="package://tactile_glove_display/meshes/f45phalanx3.dae" />
 	</geometry>
       </visual>
@@ -368,5 +368,5 @@
           <origin xyz="-0.00 -0.00 0.00" rpy="0 0 0" />
 	<geometry>
-          <mesh filename="package://tactile_glove/meshes/f45phalanx3.dae" />
+          <mesh filename="package://tactile_glove_display/meshes/f45phalanx3.dae" />
 	</geometry>
       </collision>
@@ -417,11 +417,11 @@
 	<origin xyz="-0.00 -0.00 0.00" rpy="0 0 0" />
 	<geometry>
-          <mesh filename="package://tactile_glove/meshes/f5phalanx1.dae" />
-	</geometry>
-      </visual>
-      <collision>
-	<origin xyz="-0.00 -0.00 0.00" rpy="0 0 0" />
-	<geometry>
-          <mesh filename="package://tactile_glove/meshes/f5phalanx1.dae" />
+          <mesh filename="package://tactile_glove_display/meshes/f5phalanx1.dae" />
+	</geometry>
+      </visual>
+      <collision>
+	<origin xyz="-0.00 -0.00 0.00" rpy="0 0 0" />
+	<geometry>
+          <mesh filename="package://tactile_glove_display/meshes/f5phalanx1.dae" />
 	</geometry>
       </collision>
@@ -434,5 +434,5 @@
 	<origin xyz="-0.00 -0.00 0.00" rpy="0 0 0" />
 	<geometry>
-          <mesh filename="package://tactile_glove/meshes/f5phalanx2.dae" />
+          <mesh filename="package://tactile_glove_display/meshes/f5phalanx2.dae" />
 	</geometry>
       </visual>
@@ -440,5 +440,5 @@
           <origin xyz="-0.00 -0.00 0.00" rpy="0 0 0" />
 	<geometry>
-          <mesh filename="package://tactile_glove/meshes/f5phalanx2.dae" />
+          <mesh filename="package://tactile_glove_display/meshes/f5phalanx2.dae" />
 	</geometry>
       </collision>
@@ -451,5 +451,5 @@
 	<origin xyz="-0.00 -0.00 0.00" rpy="0 0 0" />
 	<geometry>
-          <mesh filename="package://tactile_glove/meshes/f45phalanx3.dae" />
+          <mesh filename="package://tactile_glove_display/meshes/f45phalanx3.dae" />
 	</geometry>
       </visual>
@@ -457,5 +457,5 @@
           <origin xyz="-0.00 -0.00 0.00" rpy="0 0 0" />
 	<geometry>
-          <mesh filename="package://tactile_glove/meshes/f45phalanx3.dae" />
+          <mesh filename="package://tactile_glove_display/meshes/f45phalanx3.dae" />
 	</geometry>
       </collision>

File: tactile_glove_display/urdf/puthand_oryginal.urdf.xacro (robot description, xacro)
@@ -1,6 +1,6 @@
 <?xml version="1.0"?>
 <robot xmlns:xacro="http://ros.org/wiki/xacro">
-  <xacro:include filename="$(find tactile_glove)/urdf/puthand.transmission.xacro" />
-  <xacro:include filename="$(find tactile_glove)/urdf/puthand.gazebo.xacro" />
+  <xacro:include filename="$(find tactile_glove_display)/urdf/puthand.transmission.xacro" />
+  <xacro:include filename="$(find tactile_glove_display)/urdf/puthand.gazebo.xacro" />
   <xacro:property name="cyl_radius" value="0.001" />
   <!-- Inertia parameters -->
@@ -40,5 +40,5 @@
 	<origin xyz="0 0 0.0" rpy="0 0 0" />
 	<geometry>
-          <mesh filename="package://tactile_glove/meshes/metacarpusNew.dae" />
+          <mesh filename="package://tactile_glove_display/meshes/metacarpusNew.dae" />
 	</geometry>
       </visual>
@@ -46,5 +46,5 @@
 	<origin xyz="0 0 0.0" rpy="0 0 0" />
 	<geometry>
-          <mesh filename="package://tactile_glove/meshes/metacarpusNew.dae" />
+          <mesh filename="package://tactile_glove_display/meshes/metacarpusNew.dae" />
 	</geometry>
       </collision>
@@ -58,5 +58,5 @@
 	<origin xyz="0 0 0" rpy="0 0 0" />
 	<geometry>
-          <mesh filename="package://tactile_glove/meshes/metacarpal.dae" />
+          <mesh filename="package://tactile_glove_display/meshes/metacarpal.dae" />
 	</geometry>
       </visual>
@@ -64,5 +64,5 @@
 	<origin xyz="0 0 0" rpy="0 0 0" />
 	<geometry>
-          <mesh filename="package://tactile_glove/meshes/metacarpal.dae" />
+          <mesh filename="package://tactile_glove_display/meshes/metacarpal.dae" />
 	</geometry>
       </collision>
@@ -75,5 +75,5 @@
 	<origin xyz="0 0 0" rpy="0 0 0" />
 	<geometry>
-          <mesh filename="package://tactile_glove/meshes/thumbProximal.dae" />
+          <mesh filename="package://tactile_glove_display/meshes/thumbProximal.dae" />
 	</geometry>
       </visual>
@@ -81,5 +81,5 @@
           <origin xyz="0 0 0" rpy="0 0 0" />
 	<geometry>
-          <mesh filename="package://tactile_glove/meshes/thumbProximal.dae" />
+          <mesh filename="package://tactile_glove_display/meshes/thumbProximal.dae" />
 	</geometry>
       </collision>
@@ -92,5 +92,5 @@
 	<origin xyz="0 0 0" rpy="0 0 -1.5708" />
 	<geometry>
-          <mesh filename="package://tactile_glove/meshes/thumbDistal.dae" />
+          <mesh filename="package://tactile_glove_display/meshes/thumbDistal.dae" />
 	</geometry>
       </visual>
@@ -98,5 +98,5 @@
           <origin xyz="0 0 0" rpy="0 0 -1.5708" />
 	<geometry>
-          <mesh filename="package://tactile_glove/meshes/thumbDistal.dae" />
+          <mesh filename="package://tactile_glove_display/meshes/thumbDistal.dae" />
 	</geometry>
       </collision>
@@ -149,11 +149,11 @@
 	<origin xyz="-0.00 -0.00 0.00" rpy="0 0 0" />
 	<geometry>
-          <mesh filename="package://tactile_glove/meshes/fingerProximal.dae" />
-	</geometry>
-      </visual>
-      <collision>
-	<origin xyz="-0.00 -0.00 0.00" rpy="0 0 0" />
-	<geometry>
-          <mesh filename="package://tactile_glove/meshes/fingerProximal.dae" />
+          <mesh filename="package://tactile_glove_display/meshes/fingerProximal.dae" />
+	</geometry>
+      </visual>
+      <collision>
+	<origin xyz="-0.00 -0.00 0.00" rpy="0 0 0" />
+	<geometry>
+          <mesh filename="package://tactile_glove_display/meshes/fingerProximal.dae" />
 	</geometry>
       </collision>
@@ -166,5 +166,5 @@
 	<origin xyz="-0.00 -0.00 0.00" rpy="0 0 1.5708" />
 	<geometry>
-          <mesh filename="package://tactile_glove/meshes/fingerMiddle.dae" />
+          <mesh filename="package://tactile_glove_display/meshes/fingerMiddle.dae" />
 	</geometry>
       </visual>
@@ -172,5 +172,5 @@
           <origin xyz="-0.00 -0.00 0.00" rpy="0 0 1.5708" />
 	<geometry>
-          <mesh filename="package://tactile_glove/meshes/fingerMiddle.dae" />
+          <mesh filename="package://tactile_glove_display/meshes/fingerMiddle.dae" />
 	</geometry>
       </collision>
@@ -183,5 +183,5 @@
 	<origin xyz="-0.00 -0.00 0.00" rpy="0 0 0" />
 	<geometry>
-          <mesh filename="package://tactile_glove/meshes/fingerDistal.dae" />
+          <mesh filename="package://tactile_glove_display/meshes/fingerDistal.dae" />
 	</geometry>
       </visual>
@@ -189,5 +189,5 @@
           <origin xyz="-0.00 -0.0 0.00" rpy="0 0 0" />
 	<geometry>
-          <mesh filename="package://tactile_glove/meshes/fingerDistal.dae" />
+          <mesh filename="package://tactile_glove_display/meshes/fingerDistal.dae" />
 	</geometry>
       </collision>
@@ -240,11 +240,11 @@
 	<origin xyz="-0.00 -0.00 0.00" rpy="0 0 0" />
 	<geometry>
-          <mesh filename="package://tactile_glove/meshes/fingerProximal.dae" />
-	</geometry>
-      </visual>
-      <collision>
-	<origin xyz="-0.00 -0.00 0.00" rpy="0 0 0" />
-	<geometry>
-          <mesh filename="package://tactile_glove/meshes/fingerProximal.dae" />
+          <mesh filename="package://tactile_glove_display/meshes/fingerProximal.dae" />
+	</geometry>
+      </visual>
+      <collision>
+	<origin xyz="-0.00 -0.00 0.00" rpy="0 0 0" />
+	<geometry>
+          <mesh filename="package://tactile_glove_display/meshes/fingerProximal.dae" />
 	</geometry>
       </collision>
@@ -257,5 +257,5 @@
 	<origin xyz="-0.00 -0.00 0.00" rpy="0 0 1.5708" />
 	<geometry>
-          <mesh filename="package://tactile_glove/meshes/fingerMiddle.dae" />
+          <mesh filename="package://tactile_glove_display/meshes/fingerMiddle.dae" />
 	</geometry>
       </visual>
@@ -263,5 +263,5 @@
           <origin xyz="-0.00 -0.00 0.00" rpy="0 0 1.5708" />
 	<geometry>
-          <mesh filename="package://tactile_glove/meshes/fingerMiddle.dae" />
+          <mesh filename="package://tactile_glove_display/meshes/fingerMiddle.dae" />
 	</geometry>
       </collision>
@@ -274,5 +274,5 @@
 	<origin xyz="-0.00 -0.00 0.00" rpy="0 0 0" />
 	<geometry>
-          <mesh filename="package://tactile_glove/meshes/fingerDistal.dae" />
+          <mesh filename="package://tactile_glove_display/meshes/fingerDistal.dae" />
 	</geometry>
       </visual>
@@ -280,5 +280,5 @@
           <origin xyz="-0.00 -0.00 0.00" rpy="0 0 0" />
 	<geometry>
-          <mesh filename="package://tactile_glove/meshes/fingerDistal.dae" />
+          <mesh filename="package://tactile_glove_display/meshes/fingerDistal.dae" />
 	</geometry>
       </collision>
@@ -328,11 +328,11 @@
 	<origin xyz="-0.00 -0.00 0.00" rpy="0 0 0" />
 	<geometry>
-          <mesh filename="package://tactile_glove/meshes/f4phalanx1.dae" />
-	</geometry>
-      </visual>
-      <collision>
-	<origin xyz="-0.00 -0.00 0.00" rpy="0 0 0" />
-	<geometry>
-          <mesh filename="package://tactile_glove/meshes/f4phalanx1.dae" />
+          <mesh filename="package://tactile_glove_display/meshes/f4phalanx1.dae" />
+	</geometry>
+      </visual>
+      <collision>
+	<origin xyz="-0.00 -0.00 0.00" rpy="0 0 0" />
+	<geometry>
+          <mesh filename="package://tactile_glove_display/meshes/f4phalanx1.dae" />
 	</geometry>
       </collision>
@@ -345,5 +345,5 @@
 	<origin xyz="-0.00 -0.00 0.00" rpy="0 0 0" />
 	<geometry>
-          <mesh filename="package://tactile_glove/meshes/f4phalanx2.dae" />
+          <mesh filename="package://tactile_glove_display/meshes/f4phalanx2.dae" />
 	</geometry>
       </visual>
@@ -351,5 +351,5 @@
           <origin xyz="-0.00 -0.00 0.00" rpy="0 0 0" />
 	<geometry>
-          <mesh filename="package://tactile_glove/meshes/f4phalanx2.dae" />
+          <mesh filename="package://tactile_glove_display/meshes/f4phalanx2.dae" />
 	</geometry>
       </collision>
@@ -362,5 +362,5 @@
 	<origin xyz="-0.00 -0.00 0.00" rpy="0 0 0" />
 	<geometry>
-          <mesh filename="package://tactile_glove/meshes/f45phalanx3.dae" />
+          <mesh filename="package://tactile_glove_display/meshes/f45phalanx3.dae" />
 	</geometry>
       </visual>
@@ -368,5 +368,5 @@
           <origin xyz="-0.00 -0.00 0.00" rpy="0 0 0" />
 	<geometry>
-          <mesh filename="package://tactile_glove/meshes/f45phalanx3.dae" />
+          <mesh filename="package://tactile_glove_display/meshes/f45phalanx3.dae" />
 	</geometry>
       </collision>
@@ -417,11 +417,11 @@
 	<origin xyz="-0.00 -0.00 0.00" rpy="0 0 0" />
 	<geometry>
-          <mesh filename="package://tactile_glove/meshes/f5phalanx1.dae" />
-	</geometry>
-      </visual>
-      <collision>
-	<origin xyz="-0.00 -0.00 0.00" rpy="0 0 0" />
-	<geometry>
-          <mesh filename="package://tactile_glove/meshes/f5phalanx1.dae" />
+          <mesh filename="package://tactile_glove_display/meshes/f5phalanx1.dae" />
+	</geometry>
+      </visual>
+      <collision>
+	<origin xyz="-0.00 -0.00 0.00" rpy="0 0 0" />
+	<geometry>
+          <mesh filename="package://tactile_glove_display/meshes/f5phalanx1.dae" />
 	</geometry>
       </collision>
@@ -434,5 +434,5 @@
 	<origin xyz="-0.00 -0.00 0.00" rpy="0 0 0" />
 	<geometry>
-          <mesh filename="package://tactile_glove/meshes/f5phalanx2.dae" />
+          <mesh filename="package://tactile_glove_display/meshes/f5phalanx2.dae" />
 	</geometry>
       </visual>
@@ -440,5 +440,5 @@
           <origin xyz="-0.00 -0.00 0.00" rpy="0 0 0" />
 	<geometry>
-          <mesh filename="package://tactile_glove/meshes/f5phalanx2.dae" />
+          <mesh filename="package://tactile_glove_display/meshes/f5phalanx2.dae" />
 	</geometry>
       </collision>
@@ -451,5 +451,5 @@
 	<origin xyz="-0.00 -0.00 0.00" rpy="0 0 0" />
 	<geometry>
-          <mesh filename="package://tactile_glove/meshes/f45phalanx3.dae" />
+          <mesh filename="package://tactile_glove_display/meshes/f45phalanx3.dae" />
 	</geometry>
       </visual>
@@ -457,5 +457,5 @@
           <origin xyz="-0.00 -0.00 0.00" rpy="0 0 0" />
 	<geometry>
-          <mesh filename="package://tactile_glove/meshes/f45phalanx3.dae" />
+          <mesh filename="package://tactile_glove_display/meshes/f45phalanx3.dae" />
 	</geometry>
       </collision>
